Commit message: Changed urdf to xacro & Added multi_bot_launch

File: my_bot_sim/urdf/bot.urdf.xacro (robot description, xacro)
@@ -1,4 +1,5 @@
 <?xml version="1.0"?>
-<robot name="bot">
+<robot name="robot" xmlns:xacro="http://www.ros.org/wiki/xacro">
+  <xacro:arg name="robot_name" default="bot1"/>
   <!-- Materials -->
   <material name="grey">
@@ -12,6 +13,6 @@
   </material>
   <!-- Base -->
-  <link name="base_footprint"/>
-  <link name="base_link">
+  <link name="$(arg robot_name)_base_footprint"/>
+  <link name="$(arg robot_name)_base_link">
     <visual>
       <geometry>
@@ -33,5 +34,5 @@
   </link>
   <!-- Wheels -->
-  <link name="leftwheel">
+  <link name="$(arg robot_name)_leftwheel">
     <visual>
       <geometry>
@@ -46,10 +47,4 @@
       </geometry>
       <origin xyz="0 0 0" rpy="1.5708 0 0"/>
-      <gazebo>
-        <mu1>1.0</mu1>
-        <mu2>1.0</mu2>
-        <kp>100000.0</kp>
-        <kd>1.0</kd>
-      </gazebo>
     </collision>
     <inertial>
@@ -58,5 +53,5 @@
     </inertial>
   </link>
-  <link name="rightwheel">
+  <link name="$(arg robot_name)_rightwheel">
     <visual>
       <geometry>
@@ -71,10 +66,4 @@
         </geometry>
         <origin xyz="0 0 0" rpy="1.5708 0 0"/>
-        <gazebo>
-            <mu1>1.0</mu1>
-            <mu2>1.0</mu2>
-            <kp>100000.0</kp>
-            <kd>1.0</kd>
-        </gazebo>
     </collision>
     <inertial>
@@ -83,5 +72,5 @@
     </inertial>
   </link>
-  <link name="casterwheel">
+  <link name="$(arg robot_name)_casterwheel">
     <visual>
       <geometry>
@@ -102,30 +91,28 @@
   </link>
   <!-- Joints -->
-  <joint name="base_joint" type="fixed">
-    <parent link="base_footprint"/>
-    <child link="base_link"/>
+  <joint name="$(arg robot_name)_base_joint" type="fixed">
+    <parent link="$(arg robot_name)_base_footprint"/>
+    <child link="$(arg robot_name)_base_link"/>
     <origin xyz="0 0 0.1" rpy="0 0 0"/>
   </joint>
-  <joint name="leftwheel_joint" type="continuous">
-    <parent link="base_link"/>
-    <child link="leftwheel"/>
+  <joint name="$(arg robot_name)_leftwheel_joint" type="continuous">
+    <parent link="$(arg robot_name)_base_link"/>
+    <child link="$(arg robot_name)_leftwheel"/>
     <origin xyz="-0.15 0.225 0.0" rpy="0 0 0"/>
     <axis xyz="0 -1 0"/>
-    <dynamics damping="0.5" friction="1.0"/>
   </joint>
-  <joint name="rightwheel_joint" type="continuous">
-    <parent link="base_link"/>
-    <child link="rightwheel"/>
+  <joint name="$(arg robot_name)_rightwheel_joint" type="continuous">
+    <parent link="$(arg robot_name)_base_link"/>
+    <child link="$(arg robot_name)_rightwheel"/>
     <origin xyz="-0.15 -0.225 0.0" rpy="0 0 0"/>
     <axis xyz="0 -1 0"/>
-    <dynamics damping="0.5" friction="1.0"/>
   </joint>
-  <joint name="basecaster" type="fixed">
-    <parent link="base_link"/>
-    <child link="casterwheel"/>
+  <joint name="$(arg robot_name)_basecaster" type="fixed">
+    <parent link="$(arg robot_name)_base_link"/>
+    <child link="$(arg robot_name)_casterwheel"/>
     <origin xyz="0.2 0.0 -0.05" rpy="0 0 0"/>
   </joint>
   <!-- Lidar -->
-  <link name="lidar">
+  <link name="$(arg robot_name)_lidar">
     <visual>
       <geometry>
@@ -136,7 +123,7 @@
     </visual>
   </link>
-  <joint name="base_lidar_joint" type="fixed">
-    <parent link="base_link"/>
-    <child link="lidar"/>
+  <joint name="$(arg robot_name)_base_lidar_joint" type="fixed">
+    <parent link="$(arg robot_name)_base_link"/>
+    <child link="$(arg robot_name)_lidar"/>
     <origin xyz="0 0 0.225" rpy="0 0 0"/>
   </joint>
@@ -144,15 +131,14 @@
   <gazebo>
     <plugin name="diff_drive_controller" filename="libgazebo_ros_diff_drive.so">
-      <ros>
-        <remapping>cmd_vel:=/cmd_vel</remapping>
-      </ros>
       <update_rate>100.0</update_rate>
-      <left_joint>rightwheel_joint</left_joint>
-      <right_joint>leftwheel_joint</right_joint>
+      <left_joint>$(arg robot_name)_rightwheel_joint</left_joint>
+      <right_joint>$(arg robot_name)_leftwheel_joint</right_joint>
       <wheel_separation>0.45</wheel_separation>
       <wheel_diameter>0.2</wheel_diameter>
       <torque>15</torque>
       <command_topic>cmd_vel</command_topic>
+      <robot_base_frame>$(arg robot_name)_base_footprint</robot_base_frame>
       <cmd_vel_timeout>0.25</cmd_vel_timeout>
+      <publish_wheel_tf>true</publish_wheel_tf>
     </plugin>
   </gazebo>
